File: power_supply/plus_minus_12v.sch (KiCad schematic (older format))
At the start: 28 parts, among them P1 CONN_01X03, P2 CONN_01X03, T1 MYRRA-TRANSF, U1 LM317T, U2 LM337T

Commit message: power supply update
Parts:
- C1, C2, C3, C4: footprint (none) -> Capacitors_ThroughHole:C_Radial_D16_L30_P7.5
- C10, C9: footprint (none) -> Capacitors_ThroughHole:C_Radial_D5_L11_P2
- C5, C6, C7, C8: footprint (none) -> Capacitors_ThroughHole:C_Rect_L4_W2.5_P2.5
- D1, D2, D3, D4, D5, D6: footprint (none) -> Discret:DO-35
- F1: footprint (none) -> Capacitors_ThroughHole:C_Disc_D6_P5
- R1, R2: footprint (none) -> Resistors_Universal:Resistor_SMD+THTuniversal_2512_RM10_HandSoldering
- R3, R4, R5, R6: footprint (none) -> Resistors_Universal:Resistor_SMD+THTuniversal_0805to1206_RM10_HandSoldering
- U1, U2: footprint TO-220 -> TO_SOT_Packages_THT:TO-220_Neutral123_Vertical
Connections:
- net at C9.1, D3.2 (A), D5.1 (K)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: now also C7.1
Changed lines of the file:
@@
 F 0 "D1" H 3050 3250 50  0000 C CNN
 F 1 "1N4004" H 3050 3050 50  0000 C CNN
-F 2 "" H 3050 3150 50  0000 C CNN
+F 2 "Discret:DO-35" H 3050 3150 50  0001 C CNN
 F 3 "" H 3050 3150 50  0000 C CNN
 	1    3050 3150
@@
 F 0 "D2" H 3050 4350 50  0000 C CNN
 F 1 "1N4004" H 3050 4150 50  0000 C CNN
-F 2 "" H 3050 4250 50  0000 C CNN
+F 2 "Discret:DO-35" H 3050 4250 50  0001 C CNN
 F 3 "" H 3050 4250 50  0000 C CNN
 	1    3050 4250
@@
 F 0 "C1" H 3525 3400 50  0000 L CNN
 F 1 "2200uF" H 3525 3200 50  0000 L CNN
-F 2 "" H 3538 3150 50  0000 C CNN
+F 2 "Capacitors_ThroughHole:C_Radial_D16_L30_P7.5" H 3538 3150 50  0001 C CNN
 F 3 "" H 3500 3300 50  0000 C CNN
 	1    3500 3300
@@
 F 0 "C2" H 3525 4200 50  0000 L CNN
 F 1 "2200uF" H 3525 4000 50  0000 L CNN
-F 2 "" H 3538 3950 50  0000 C CNN
+F 2 "Capacitors_ThroughHole:C_Radial_D16_L30_P7.5" H 3538 3950 50  0001 C CNN
 F 3 "" H 3500 4100 50  0000 C CNN
 	1    3500 4100
@@
 F 0 "R1" V 4030 3000 50  0000 C CNN
 F 1 "4R7" V 3850 3000 50  0000 C CNN
-F 2 "" V 3880 3000 50  0000 C CNN
+F 2 "Resistors_Universal:Resistor_SMD+THTuniversal_2512_RM10_HandSoldering" V 3880 3000 50  0001 C CNN
 F 3 "" H 3950 3000 50  0000 C CNN
 	1    3950 3000
@@
 F 0 "R2" V 4030 4400 50  0000 C CNN
 F 1 "4R7" V 3850 4400 50  0000 C CNN
-F 2 "" V 3880 4400 50  0000 C CNN
+F 2 "Resistors_Universal:Resistor_SMD+THTuniversal_2512_RM10_HandSoldering" V 3880 4400 50  0001 C CNN
 F 3 "" H 3950 4400 50  0000 C CNN
 	1    3950 4400
@@
 F 0 "C4" H 4375 4200 50  0000 L CNN
 F 1 "2200uF" H 4375 4000 50  0000 L CNN
-F 2 "" H 4388 3950 50  0000 C CNN
+F 2 "Capacitors_ThroughHole:C_Radial_D16_L30_P7.5" H 4388 3950 50  0001 C CNN
 F 3 "" H 4350 4100 50  0000 C CNN
 	1    4350 4100
@@
 F 0 "C3" H 4375 3400 50  0000 L CNN
 F 1 "2200uF" H 4375 3200 50  0000 L CNN
-F 2 "" H 4388 3150 50  0000 C CNN
+F 2 "Capacitors_ThroughHole:C_Radial_D16_L30_P7.5" H 4388 3150 50  0001 C CNN
 F 3 "" H 4350 3300 50  0000 C CNN
 	1    4350 3300
@@
 F 0 "C5" H 4825 3400 50  0000 L CNN
 F 1 "100nF" H 4825 3200 50  0000 L CNN
-F 2 "" H 4838 3150 50  0000 C CNN
+F 2 "Capacitors_ThroughHole:C_Rect_L4_W2.5_P2.5" H 4838 3150 50  0001 C CNN
 F 3 "" H 4800 3300 50  0000 C CNN
 	1    4800 3300
@@
 F 0 "C6" H 4825 4200 50  0000 L CNN
 F 1 "100nF" H 4825 4000 50  0000 L CNN
-F 2 "" H 4838 3950 50  0000 C CNN
+F 2 "Capacitors_ThroughHole:C_Rect_L4_W2.5_P2.5" H 4838 3950 50  0001 C CNN
 F 3 "" H 4800 4100 50  0000 C CNN
 	1    4800 4100
@@
 F 0 "U1" H 5400 3250 50  0000 C CNN
 F 1 "LM317T" H 5600 3250 50  0000 L CNN
-F 2 "TO-220" H 5600 3150 50  0000 C CIN
+F 2 "TO_SOT_Packages_THT:TO-220_Neutral123_Vertical" H 5600 3150 50  0001 C CIN
 F 3 "" H 5600 3050 50  0000 C CNN
 	1    5600 3050
@@
 F 0 "U2" H 5400 4150 50  0000 C CNN
 F 1 "LM337T" H 5600 4150 50  0000 L CNN
-F 2 "TO-220" H 5600 4250 50  0000 C CIN
+F 2 "TO_SOT_Packages_THT:TO-220_Neutral123_Vertical" H 5600 4250 50  0001 C CIN
 F 3 "" H 5600 4350 50  0000 C CNN
 	1    5600 4350
@@
 F 0 "R3" V 6380 3150 50  0000 C CNN
 F 1 "330R" V 6200 3150 50  0000 C CNN
-F 2 "" V 6230 3150 50  0000 C CNN
+F 2 "Resistors_Universal:Resistor_SMD+THTuniversal_0805to1206_RM10_HandSoldering" V 6230 3150 50  0001 C CNN
 F 3 "" H 6300 3150 50  0000 C CNN
 	1    6300 3150
@@
 F 0 "R6" V 6380 4250 50  0000 C CNN
 F 1 "330R" V 6200 4250 50  0000 C CNN
-F 2 "" V 6230 4250 50  0000 C CNN
+F 2 "Resistors_Universal:Resistor_SMD+THTuniversal_0805to1206_RM10_HandSoldering" V 6230 4250 50  0001 C CNN
 F 3 "" H 6300 4250 50  0000 C CNN
 	1    6300 4250
@@
 F 0 "R5" V 6380 3900 50  0000 C CNN
 F 1 "2K7" V 6200 3900 50  0000 C CNN
-F 2 "" V 6230 3900 50  0000 C CNN
+F 2 "Resistors_Universal:Resistor_SMD+THTuniversal_0805to1206_RM10_HandSoldering" V 6230 3900 50  0001 C CNN
 F 3 "" H 6300 3900 50  0000 C CNN
 	1    6300 3900
@@
 F 0 "R4" V 6380 3500 50  0000 C CNN
 F 1 "2K7" V 6200 3500 50  0000 C CNN
-F 2 "" V 6230 3500 50  0000 C CNN
+F 2 "Resistors_Universal:Resistor_SMD+THTuniversal_0805to1206_RM10_HandSoldering" V 6230 3500 50  0001 C CNN
 F 3 "" H 6300 3500 50  0000 C CNN
 	1    6300 3500
@@
 F 0 "C7" H 6825 3400 50  0000 L CNN
 F 1 "100nF" H 6825 3200 50  0000 L CNN
-F 2 "" H 6838 3150 50  0000 C CNN
+F 2 "Capacitors_ThroughHole:C_Rect_L4_W2.5_P2.5" H 6838 3150 50  0001 C CNN
 F 3 "" H 6800 3300 50  0000 C CNN
 	1    6800 3300
@@
 	3500 3000 3500 3150
 $Comp
-L GND #PWR2
+L GND #PWR01
 U 1 1 57D49C22
 P 3950 3850
-F 0 "#PWR2" H 3950 3600 50  0001 C CNN
+F 0 "#PWR01" H 3950 3600 50  0001 C CNN
 F 1 "GND" H 3950 3700 50  0000 C CNN
 F 2 "" H 3950 3850 50  0000 C CNN
@@
 F 0 "C8" H 6825 4200 50  0000 L CNN
 F 1 "100nF" H 6825 4000 50  0000 L CNN
-F 2 "" H 6838 3950 50  0000 C CNN
+F 2 "Capacitors_ThroughHole:C_Rect_L4_W2.5_P2.5" H 6838 3950 50  0001 C CNN
 F 3 "" H 6800 4100 50  0000 C CNN
 	1    6800 4100
@@
 F 0 "D5" H 7250 3400 50  0000 C CNN
 F 1 "1N4004" H 7250 3200 50  0000 C CNN
-F 2 "" H 7250 3300 50  0000 C CNN
+F 2 "Discret:DO-35" H 7250 3300 50  0001 C CNN
 F 3 "" H 7250 3300 50  0000 C CNN
 	1    7250 3300
@@
 F 0 "D6" H 7250 4200 50  0000 C CNN
 F 1 "1N4004" H 7250 4000 50  0000 C CNN
-F 2 "" H 7250 4100 50  0000 C CNN
+F 2 "Discret:DO-35" H 7250 4100 50  0001 C CNN
 F 3 "" H 7250 4100 50  0000 C CNN
 	1    7250 4100
@@
 F 0 "C10" H 7775 4200 50  0000 L CNN
 F 1 "10uF" H 7775 4000 50  0000 L CNN
-F 2 "" H 7788 3950 50  0000 C CNN
+F 2 "Capacitors_ThroughHole:C_Radial_D5_L11_P2" H 7788 3950 50  0001 C CNN
 F 3 "" H 7750 4100 50  0000 C CNN
 	1    7750 4100
@@
 F 0 "C9" H 7775 3400 50  0000 L CNN
 F 1 "10uF" H 7775 3200 50  0000 L CNN
-F 2 "" H 7788 3150 50  0000 C CNN
+F 2 "Capacitors_ThroughHole:C_Radial_D5_L11_P2" H 7788 3150 50  0001 C CNN
 F 3 "" H 7750 3300 50  0000 C CNN
 	1    7750 3300
@@
 F 0 "D3" H 5600 2700 50  0000 C CNN
 F 1 "1N4004" H 5600 2500 50  0000 C CNN
-F 2 "" H 5600 2600 50  0000 C CNN
+F 2 "Discret:DO-35" H 5600 2600 50  0001 C CNN
 F 3 "" H 5600 2600 50  0000 C CNN
 	1    5600 2600
@@
 F 0 "D4" H 5600 4900 50  0000 C CNN
 F 1 "1N4004" H 5600 4700 50  0000 C CNN
-F 2 "" H 5600 4800 50  0000 C CNN
+F 2 "Discret:DO-35" H 5600 4800 50  0001 C CNN
 F 3 "" H 5600 4800 50  0000 C CNN
 	1    5600 4800
@@
 	1500 3800 1850 3800
 $Comp
-L GND #PWR1
+L GND #PWR02
 U 1 1 57D5AF7E
 P 1700 3400
-F 0 "#PWR1" H 1700 3150 50  0001 C CNN
+F 0 "#PWR02" H 1700 3150 50  0001 C CNN
 F 1 "GND" H 1700 3250 50  0000 C CNN
 F 2 "" H 1700 3400 50  0000 C CNN
@@
 F 0 "F1" H 2660 3360 50  0000 L CNN
 F 1 "F_Small" H 2580 3240 50  0000 L CNN
-F 2 "" H 2700 3300 50  0000 C CNN
+F 2 "Capacitors_ThroughHole:C_Disc_D6_P5" H 2700 3300 50  0001 C CNN
 F 3 "" H 2700 3300 50  0000 C CNN
 	1    2700 3300
@@
 Wire Wire Line
 	2600 3300 2500 3300
+Connection ~ 6800 3000
 $EndSCHEMATC

Commit message: New transformer footprint, updated power PCB
Parts:
- T1: footprint Transformers_CHK:Trafo_CHK-EI42-5VA_1xSec -> My Shit:Transformer-5VA_1xSec
Changed lines of the file:
@@
 F 0 "T1" H 2150 3900 50  0000 C CNN
 F 1 "MYRRA-TRANSF" H 2150 3100 50  0000 C CNN
-F 2 "Transformers_CHK:Trafo_CHK-EI42-5VA_1xSec" H 2150 3500 50  0001 C CNN
+F 2 "My Shit:Transformer-5VA_1xSec" H 2150 3500 50  0001 C CNN
 F 3 "" H 2150 3500 50  0000 C CNN
 	1    2150 3500
