File: stepper_generator/generator.kicad_pcb (KiCad board)
At the start: 2 copper layers, 54.6 x 21.6 mm, 26 parts, among them J1 USB_A, J2 Screw_Terminal_01x02, J4 Conn_01x02_Male, J5 Conn_01x04_Male, U1 TPS2514, U2 LM317_3PinPackage

Commit message: Modify the USB A female footprint to comply with OSHpark settings
Parts:
- moved J1 0.09 mm to (65.5, 64.2)
Changed lines of the file:
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@@
-    )
-  )
-  (module my_shit:USB_A_Female (layer F.Cu)
-    (at 65.405 64.135 180)
-    (descr http://cnctech.us/pdfs/1001-011-01101.pdf)
-    (tags USB-A)
-    (attr smd)
-    (fp_text reference J1 (at -4.445 3.175 180) (layer F.SilkS)
-      (effects (font (size 1 1) (thickness 0.15)))
-    )
-    (fp_text value USB_A (at 0 8) (layer F.Fab) hide
-      (effects (font (size 1 1) (thickness 0.15)))
-    )
-    (fp_line (start -7.9 6.025) (end -7.9 -6.025) (layer F.Fab) (width 0.1))
-    (fp_line (start -7.9 -6.025) (end 10.9 -6.025) (layer F.Fab) (width 0.1))
-    (fp_line (start -7.9 6.025) (end 10.9 6.025) (layer F.Fab) (width 0.1))
-    (fp_line (start 10.9 6.025) (end 10.9 -6.025) (layer F.Fab) (width 0.1))
-    (fp_line (start -10.4 3.75) (end -10.4 3.25) (layer F.Fab) (width 0.1))
-    (fp_line (start -10.4 3.25) (end -7.9 3.25) (layer F.Fab) (width 0.1))
-    (fp_line (start -10.4 3.75) (end -7.9 3.75) (layer F.Fab) (width 0.1))
-    (fp_line (start -10.4 0.75) (end -7.9 0.75) (layer F.Fab) (width 0.1))
-    (fp_line (start -10.4 1.25) (end -10.4 0.75) (layer F.Fab) (width 0.1))
-    (fp_line (start -10.4 1.25) (end -7.9 1.25) (layer F.Fab) (width 0.1))
-    (fp_line (start -10.4 -0.75) (end -10.4 -1.25) (layer F.Fab) (width 0.1))
-    (fp_line (start -10.4 -0.75) (end -7.9 -0.75) (layer F.Fab) (width 0.1))
-    (fp_line (start -10.4 -1.25) (end -7.9 -1.25) (layer F.Fab) (width 0.1))
-    (fp_line (start -10.4 -3.75) (end -7.9 -3.75) (layer F.Fab) (width 0.1))
-    (fp_line (start -10.4 -3.25) (end -10.4 -3.75) (layer F.Fab) (width 0.1))
-    (fp_line (start -10.4 -3.25) (end -7.9 -3.25) (layer F.Fab) (width 0.1))
-    (fp_line (start -8.02 -4.4) (end -8.02 4.4) (layer F.SilkS) (width 0.12))
-    (fp_line (start -1.016 6.025) (end -1.016 -6.025) (layer Dwgs.User) (width 0.1))
-    (fp_text user "PCB Edge" (at -1.524 -0.05 270) (layer Dwgs.User)
-      (effects (font (size 0.6 0.6) (thickness 0.09)))
-    )
-    (fp_line (start -4.85 -6.145) (end -3.8 -6.145) (layer F.SilkS) (width 0.12))
-    (fp_line (start -4.85 6.145) (end -3.8 6.145) (layer F.SilkS) (width 0.12))
-    (fp_line (start -11.4 6.35) (end -11.4 -6.35) (layer F.CrtYd) (width 0.05))
-    (fp_line (start -11.4 -6.35) (end -9.15 -6.35) (layer F.CrtYd) (width 0.05))
-    (fp_line (start -9.15 -7.15) (end -9.15 -6.35) (layer F.CrtYd) (width 0.05))
-    (fp_line (start -9.15 -7.15) (end -4.65 -7.15) (layer F.CrtYd) (width 0.05))
-    (fp_line (start -4.65 -6.52) (end -4.65 -7.15) (layer F.CrtYd) (width 0.05))
-    (fp_line (start -4.65 -6.52) (end 11.4 -6.52) (layer F.CrtYd) (width 0.05))
-    (fp_line (start 11.4 6.52) (end 11.4 -6.52) (layer F.CrtYd) (width 0.05))
-    (fp_text user %R (at -6 0 270) (layer F.Fab) hide
-      (effects (font (size 1 1) (thickness 0.15)))
-    )
-    (fp_line (start -4.65 6.52) (end 11.4 6.52) (layer F.CrtYd) (width 0.05))
-    (fp_line (start -4.65 7.15) (end -4.65 6.52) (layer F.CrtYd) (width 0.05))
-    (fp_line (start -9.15 7.15) (end -4.65 7.15) (layer F.CrtYd) (width 0.05))
-    (fp_line (start -9.15 6.35) (end -9.15 7.15) (layer F.CrtYd) (width 0.05))
-    (fp_line (start -11.4 6.35) (end -9.15 6.35) (layer F.CrtYd) (width 0.05))
-    (pad 2 thru_hole circle (at -9.65 -1 180) (size 1.5 1.5) (drill 0.8) (layers *.Cu *.Mask)
-      (net 9 "Net-(J1-Pad2)"))
-    (pad 3 thru_hole circle (at -9.65 1 180) (size 1.5 1.5) (drill 0.8) (layers *.Cu *.Mask)
-      (net 10 "Net-(J1-Pad3)"))
-    (pad 1 thru_hole circle (at -9.65 -3.5 180) (size 2 2) (drill 0.8) (layers *.Cu *.Mask)
-      (net 1 "Net-(C1-Pad1)"))
-    (pad 4 thru_hole circle (at -9.65 3.5 180) (size 2 2) (drill 0.8) (layers *.Cu *.Mask)
-      (net 2 "Net-(C1-Pad2)"))
-    (pad 5 thru_hole oval (at -6.9 -5.7 180) (size 3.5 1.9) (drill oval 2.5 0.9) (layers *.Cu *.Mask)
-      (net 2 "Net-(C1-Pad2)"))
-    (pad 5 thru_hole oval (at -6.9 5.7 180) (size 3.5 1.9) (drill oval 2.5 0.9) (layers *.Cu *.Mask)
-      (net 2 "Net-(C1-Pad2)"))
-    (model ${KISYS3DMOD}/Connector_USB.3dshapes/USB_A_CNCTech_1001-011-01101_Horizontal.wrl
-      (at (xyz 0 0 0))
-      (scale (xyz 1 1 1))
-      (rotate (xyz 0 0 0))
     )
   )
@@
       (at (xyz 0 0 0))
       (scale (xyz 1 1 1))
+      (rotate (xyz 0 0 0))
+    )
+  )
+  (module my_shit:USB_A_Female (layer F.Cu)
+    (at 65.49 64.15 180)
+    (descr http://cnctech.us/pdfs/1001-011-01101.pdf)
+    (tags USB-A)
+    (attr smd)
+    (fp_text reference J1 (at -5.122 -0.366 180) (layer F.SilkS)
+      (effects (font (size 1 1) (thickness 0.15)))
+    )
+    (fp_text value USB_A (at 0 8) (layer F.Fab) hide
+      (effects (font (size 1 1) (thickness 0.15)))
+    )
+    (fp_line (start -7.9 6.025) (end -7.9 -6.025) (layer F.Fab) (width 0.1))
+    (fp_line (start -7.9 -6.025) (end 10.9 -6.025) (layer F.Fab) (width 0.1))
+    (fp_line (start -7.9 6.025) (end 10.9 6.025) (layer F.Fab) (width 0.1))
+    (fp_line (start 10.9 6.025) (end 10.9 -6.025) (layer F.Fab) (width 0.1))
+    (fp_line (start -10.4 3.75) (end -10.4 3.25) (layer F.Fab) (width 0.1))
+    (fp_line (start -10.4 3.25) (end -7.9 3.25) (layer F.Fab) (width 0.1))
+    (fp_line (start -10.4 3.75) (end -7.9 3.75) (layer F.Fab) (width 0.1))
+    (fp_line (start -10.4 0.75) (end -7.9 0.75) (layer F.Fab) (width 0.1))
+    (fp_line (start -10.4 1.25) (end -10.4 0.75) (layer F.Fab) (width 0.1))
+    (fp_line (start -10.4 1.25) (end -7.9 1.25) (layer F.Fab) (width 0.1))
+    (fp_line (start -10.4 -0.75) (end -10.4 -1.25) (layer F.Fab) (width 0.1))
+    (fp_line (start -10.4 -0.75) (end -7.9 -0.75) (layer F.Fab) (width 0.1))
+    (fp_line (start -10.4 -1.25) (end -7.9 -1.25) (layer F.Fab) (width 0.1))
+    (fp_line (start -10.4 -3.75) (end -7.9 -3.75) (layer F.Fab) (width 0.1))
+    (fp_line (start -10.4 -3.25) (end -10.4 -3.75) (layer F.Fab) (width 0.1))
+    (fp_line (start -10.4 -3.25) (end -7.9 -3.25) (layer F.Fab) (width 0.1))
+    (fp_line (start -8.02 -4.4) (end -8.02 4.4) (layer F.SilkS) (width 0.12))
+    (fp_line (start -1.016 6.025) (end -1.016 -6.025) (layer Dwgs.User) (width 0.1))
+    (fp_text user "PCB Edge" (at -1.524 -0.05 270) (layer Dwgs.User)
+      (effects (font (size 0.6 0.6) (thickness 0.09)))
+    )
+    (fp_line (start -4.85 -6.145) (end -3.8 -6.145) (layer F.SilkS) (width 0.12))
+    (fp_line (start -4.85 6.145) (end -3.8 6.145) (layer F.SilkS) (width 0.12))
+    (fp_line (start -11.4 6.35) (end -11.4 -6.35) (layer F.CrtYd) (width 0.05))
+    (fp_line (start -11.4 -6.35) (end -9.15 -6.35) (layer F.CrtYd) (width 0.05))
+    (fp_line (start -9.15 -7.15) (end -9.15 -6.35) (layer F.CrtYd) (width 0.05))
+    (fp_line (start -9.15 -7.15) (end -4.65 -7.15) (layer F.CrtYd) (width 0.05))
+    (fp_line (start -4.65 -6.52) (end -4.65 -7.15) (layer F.CrtYd) (width 0.05))
+    (fp_line (start -4.65 -6.52) (end 11.4 -6.52) (layer F.CrtYd) (width 0.05))
+    (fp_line (start 11.4 6.52) (end 11.4 -6.52) (layer F.CrtYd) (width 0.05))
+    (fp_text user %R (at -6 0 270) (layer F.Fab) hide
+      (effects (font (size 1 1) (thickness 0.15)))
+    )
+    (fp_line (start -4.65 6.52) (end 11.4 6.52) (layer F.CrtYd) (width 0.05))
+    (fp_line (start -4.65 7.15) (end -4.65 6.52) (layer F.CrtYd) (width 0.05))
+    (fp_line (start -9.15 7.15) (end -4.65 7.15) (layer F.CrtYd) (width 0.05))
+    (fp_line (start -9.15 6.35) (end -9.15 7.15) (layer F.CrtYd) (width 0.05))
+    (fp_line (start -11.4 6.35) (end -9.15 6.35) (layer F.CrtYd) (width 0.05))
+    (pad 2 thru_hole circle (at -9.65 -1 180) (size 1.5 1.5) (drill 0.8) (layers *.Cu *.Mask)
+      (net 9 "Net-(J1-Pad2)"))
+    (pad 3 thru_hole circle (at -9.65 1 180) (size 1.5 1.5) (drill 0.8) (layers *.Cu *.Mask)
+      (net 10 "Net-(J1-Pad3)"))
+    (pad 1 thru_hole circle (at -9.65 -3.5 180) (size 2 2) (drill 0.8) (layers *.Cu *.Mask)
+      (net 1 "Net-(C1-Pad1)"))
+    (pad 4 thru_hole circle (at -9.65 3.5 180) (size 2 2) (drill 0.8) (layers *.Cu *.Mask)
+      (net 2 "Net-(C1-Pad2)"))
+    (pad 5 thru_hole circle (at -6.9 -5.7 180) (size 3.5 3.5) (drill 2.5) (layers *.Cu *.Mask)
+      (net 2 "Net-(C1-Pad2)"))
+    (pad 5 thru_hole circle (at -6.9 5.7 180) (size 3.5 3.5) (drill 2.5) (layers *.Cu *.Mask)
+      (net 2 "Net-(C1-Pad2)"))
+    (model ${KISYS3DMOD}/Connector_USB.3dshapes/USB_A_CNCTech_1001-011-01101_Horizontal.wrl
+      (at (xyz 0 0 0))
+      (scale (xyz 1 1 1))

Commit message: Flip the USB connector on the stepper generator
Parts:
- moved J1 0.12 mm to (65.5, 64.3)
Routing:
- net Net-(J1-Pad3): track 3.82 -> 6.21 mm, vias 0 -> 1
- net Net-(C1-Pad1): track 51.7 -> 50.6 mm
- net Net-(J1-Pad2): track 3.73 -> 3.03 mm

Commit message: Add a source text to the stepper generator board
Other:
- board text added: "github: jonronen"
Changed lines of the file:
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@@
   (general
     (thickness 1.6)
-    (drawings 9)
+    (drawings 10)
     (tracks 87)
     (zones 0)
@@
     )
   )
+  (gr_text "github:\njonronen" (at 87.63 66.04) (layer B.SilkS)
+    (effects (font (size 1.5 1.5) (thickness 0.3)) (justify mirror))
+  )
   (gr_text 0 (at 85.09 70.485) (layer F.SilkS)
