File: pseudo_reverb/pseudo_reverb.kicad_pcb (KiCad board)
At the start: 2 copper layers, 61 x 43.2 mm, 32 parts, among them U1 L7805, U2 PT2399

Commit message: Add power notations in pseudo reverb board
Other:
- board text added: "+"
- board text added: "-"
- board text added: "5V"
- board text added: "9V"
Changed lines of the file:
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@@
   (gr_line (start 121.92 134.62) (end 121.92 91.44) (layer "Edge.Cuts") (width 0.05))
   (gr_line (start 182.88 134.62) (end 121.92 134.62) (layer "Edge.Cuts") (width 0.05))
+  (gr_text "9V" (at 170.18 93.98) (layer "F.SilkS")
+    (effects (font (size 1 1) (thickness 0.15)))
+  )
+  (gr_text "+" (at 129.54 113.14 90) (layer "F.SilkS")
+    (effects (font (size 1 1) (thickness 0.15)))
+  )
+  (gr_text "+" (at 175.26 109.22 90) (layer "F.SilkS")
+    (effects (font (size 1 1) (thickness 0.15)))
+  )
+  (gr_text "-" (at 175.26 107.95 90) (layer "F.SilkS")
+    (effects (font (size 1 1) (thickness 0.15)))
+  )
+  (gr_text "+" (at 175.26 100.33 90) (layer "F.SilkS")
+    (effects (font (size 1 1) (thickness 0.15)))
+  )
+  (gr_text "-" (at 175.26 116.231 90) (layer "F.SilkS")
+    (effects (font (size 1 1) (thickness 0.15)))
+  )
+  (gr_text "5V" (at 157.48 93.98) (layer "F.SilkS")
+    (effects (font (size 1 1) (thickness 0.15)))
+  )
+  (gr_text "-" (at 129.54 107.84 90) (layer "F.SilkS")
+    (effects (font (size 1 1) (thickness 0.15)))
+  )
   (segment (start 133.35 123.19) (end 133.35 124.54) (width 0.25) (layer "F.Cu") (net 1))
   (segment (start 133.35 124.54) (end 125.81 132.08) (width 0.25) (layer "F.Cu") (net 1))
