File: tube_like_preamp/tube_like_preamp.kicad_sch (KiCad schematic)
At the start: 51 parts, among them J1 JACK_STEREO, J2 JACK_STEREO, J3 Conn_01x02, Q1 BS170, Q2 BC109, Q3 BS170, Q4 BS170, Q5 BC109, Q6 BS170

Commit message: Improve Tube-Like Preamp
Parts:
- Q2, Q5: value BC109 -> 2N5088; footprint Package_TO_SOT_THT:TO-18-3 -> Package_TO_SOT_THT:TO-92_Inline
Changed lines of the file:
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@@
 		(on_board yes)
 		(dnp no)
-		(fields_autoplaced yes)
 		(property "Reference" "Q5"
 			(at 138.43 118.1099 0)
@@
 			)
 		)
-		(property "Value" "BC109"
-			(at 138.43 120.6499 0)
-			(effects
-				(font
-					(size 1.27 1.27)
-				)
-				(justify left)
-			)
-		)
-		(property "Footprint" "Package_TO_SOT_THT:TO-18-3"
+		(property "Value" "2N5088"
+			(at 137.16 115.824 0)
+			(effects
+				(font
+					(size 1.27 1.27)
+				)
+				(justify left)
+			)
+		)
+		(property "Footprint" "Package_TO_SOT_THT:TO-92_Inline"
 			(at 138.43 121.285 0)
 			(effects
@@
 			)
 		)
-		(property "Value" "BC109"
+		(property "Value" "2N5088"
 			(at 138.43 59.6899 0)
 			(effects
@@
 			)
 		)
-		(property "Footprint" "Package_TO_SOT_THT:TO-18-3"
+		(property "Footprint" "Package_TO_SOT_THT:TO-92_Inline"
 			(at 138.43 60.325 0)
 			(effects
